Commit message: match urdf with Kelly's description

File: model/cartpole.urdf (robot description, URDF)
Before this commit: robot physics, 3 links, 2 joints
Links:
- link cart: mass 1 -> 2
- link pole: mass 10 -> 0.5; geometry collision box size=0.05 0.05 0.5; visual box size=0.05 0.05 0.5
Joints:
- joint cart_to_pole: axis 0 1 0 -> 0 -1 0; origin xyz=0.0 0.0 0 -> xyz=0.0 0.0 0 rpy=0.0 3.14159 0.0

Commit message: fix joint configuration size by changing joint type in urdf

File: model/cartpole.urdf (robot description, URDF)
Before this commit: robot physics, 3 links, 2 joints
Joints:
- joint cart_to_pole: limit (none) -> lower=-6.28318530718 upper=6.28318530718 effort=1000.0 velocity=1000.0; type continuous -> revolute
